Commit message: added joint position control and joint data stream

File: software/Nightmare_ros_code/nightmare_description/urdf/nightmare_v2.urdf (robot description, URDF)
Before this commit: robot nightmare_v2, 54 links, 53 joints
Links:
- link base_link: mass 1.536457 -> None

Commit message: fixed 3d model center position

File: software/Nightmare_ros_code/nightmare_description/urdf/nightmare_v2.urdf (robot description, URDF)
Before this commit: robot nightmare_v2, 54 links, 53 joints
Joints:
- joint Rigid14: origin xyz=0.010319 -0.059677 0.1115 rpy=0 0 0 -> xyz=-0.039681 -0.099177 0.038 rpy=0 0 0
- joint Rigid15: origin xyz=0.09251 -0.062505 0.1115 rpy=0 0 0 -> xyz=0.04251 -0.102005 0.038 rpy=0 0 0
- joint Rigid16: origin xyz=0.06025 -0.0795 0.1115 rpy=0 0 0 -> xyz=0.01025 -0.119 0.038 rpy=0 0 0
- joint Rigid17: origin xyz=0.127311 -0.005052 0.1115 rpy=0 0 0 -> xyz=0.077311 -0.044552 0.038 rpy=0 0 0
- joint Rigid18: origin xyz=0.127311 0.084052 0.1115 rpy=0 0 0 -> xyz=0.077311 0.044552 0.038 rpy=0 0 0
- joint Rigid19: origin xyz=0.09251 0.141505 0.1115 rpy=0 0 0 -> xyz=0.04251 0.102005 0.038 rpy=0 0 0
- joint Rigid20: origin xyz=0.03975 0.1585 0.1115 rpy=0 0 0 -> xyz=-0.01025 0.119 0.038 rpy=0 0 0
- joint Rigid21: origin xyz=0.00749 0.141505 0.1115 rpy=0 0 0 -> xyz=-0.04251 0.102005 0.038 rpy=0 0 0
- joint Rigid22: origin xyz=-0.027311 0.084052 0.1115 rpy=0 0 0 -> xyz=-0.077311 0.044552 0.038 rpy=0 0 0
- joint Rigid23: origin xyz=-0.027311 -0.005052 0.1115 rpy=0 0 0 -> xyz=-0.077311 -0.044552 0.038 rpy=0 0 0
